File: ModelloT.kicad_sch (KiCad schematic)
At the start: 18 parts, among them J1 ROM, J10 ACI, J11 FDC, J2 RAM2, J3 RAM0, J4 RAM1, J5 SYNC, J6 MEM, J7 US1, J8 PRT, J9 US2, U1 Z80, U10 74LS245, U15 74LS157, U3 74LS245, U6 74LS139, U7 74LS32, U8 74LS00

Commit message: completed SYNC pinout, 90% of MEM, reset circuit, beginning of ROM addressing
Parts:
- added C24: 33n, symbol Device:C
- added C25: 10u, symbol Device:C_Polarized
- added C6: .002, symbol Device:C
- added JP1: RS, symbol Jumper:Jumper_2_Bridged
- added JVID: Conn_01x02, symbol Connector_Generic:Conn_01x02
- added R3: 470, symbol Device:R
- added R4: 10k, symbol Device:R
- added U11: 74LS74, symbol 74xx:74LS74
- added U12: 74LS121, symbol 74xx:74LS121
- added U13, U9: 74LS04, symbol 74xx:74LS04
- added U14: 74LS32, symbol 74xx:74LS32
- added U16, U17: 74LS157, symbol 74xx:74LS157
- added unit 1 of U6
Connections:
- net +12V: now also J5.43 (Pin_43), J6.43 (Pin_43)
- net +5V: now also J5.40 (Pin_40), J5.41 (Pin_41), J6.40 (Pin_40), J6.41 (Pin_41), C25.1, R4.1, U11.2 (D), U11.4 (~{S}), U12.14 (VCC)
- net -5V: now also J5.42 (Pin_42), J6.42 (Pin_42), C24.1
- net A0: now also J5.23 (Pin_23)
- net A1: now also J5.21 (Pin_21)
- net A2: now also J5.19 (Pin_19)
- net A3: now also J5.17 (Pin_17)
- net A4: now also J5.15 (Pin_15)
- net A5: now also J5.13 (Pin_13), U1.35 (A_{5}), U16.2 (I0a)
- net A6: now also J5.11 (Pin_11), U15.11 (I0c)
- net A7: now also J5.9 (Pin_9), U15.5 (I0b)
- net GND: now also J5.1 (Pin_1), J5.2 (Pin_2), J5.44 (Pin_44), J5.45 (Pin_45), J6.1 (Pin_1), J6.2 (Pin_2), J6.44 (Pin_44), J6.45 (Pin_45), C24.2, R3.2, U12.3 (A1), U12.4 (A2), U12.7 (GND)
- net M1: now also U13.1
- net PHI: now also J5.27 (Pin_27)
- net d0: now also J6.27 (Pin_27)
- net d1: now also J6.29 (Pin_29)
- net d2: now also J6.23 (Pin_23)
- net d3: now also J6.17 (Pin_17)
- net d4: now also J6.15 (Pin_15)
- net d5: now also J6.19 (Pin_19)
- net d6: now also J6.21 (Pin_21)
- net d7: now also J6.25 (Pin_25)
- net ~{IORQ}: now also U11.13 (~{R})
- net ~{WR}: now also J6.33 (Pin_33)
- net A11: now reaches J1.6 (Pin_6)
- net A11: now also J6.31 (Pin_31), U1.1 (A_{11})
- net VID7: now reaches J5.10 (Pin_10)
- net VID7: now also U15.6 (I1b)
- net VID6: now reaches J5.12 (Pin_12)
- net VID6: now also U15.10 (I1c)
- net VID5: now reaches J5.14 (Pin_14)
- net VID5: now also U16.3 (I1a)
- net VID4: now reaches J5.16 (Pin_16)
- net VID3: now reaches J5.18 (Pin_18)
- net VID2: now reaches J5.20 (Pin_20)
- net VID1: now reaches J5.22 (Pin_22)
- net VID0: now reaches J5.24 (Pin_24)
- net VID0: now also U17.6 (I1b)
- net dqa11: now reaches J5.25 (Pin_25)
- net dqa11: now also J6.16 (Pin_16)
- net dqa10: now reaches J5.28 (Pin_28)
- net dqa10: now also J6.22 (Pin_22)
- net dqa9: now reaches J5.29 (Pin_29)
- net dqa9: now also J6.24 (Pin_24)
- net boh0: now reaches J5.3 (Pin_3)
- net boh0: now also J6.3 (Pin_3)
- net dqa8: now reaches J5.30 (Pin_30)
- net dqa8: now also J6.26 (Pin_26)
- net dqa7: now reaches J5.31 (Pin_31)
- net dqa7: now also J6.28 (Pin_28)
- net dqa6: now reaches J5.32 (Pin_32)
- net dqa6: now also J6.30 (Pin_30)
- net dqa5: now reaches J5.33 (Pin_33)
- net dqa5: now also J6.32 (Pin_32)
- net dqa4: now reaches J5.34 (Pin_34)
- net dqa3: now reaches J5.35 (Pin_35)
- net dqa2: now reaches J5.36 (Pin_36)
- net dqa1: now reaches J5.37 (Pin_37)
- net dqa1: now also J6.37 (Pin_37)
- net dqa0: now reaches J5.38 (Pin_38)
- net dqa0: now also J6.38 (Pin_38)
- net VSEL: now reaches J5.4 (Pin_4), J6.4 (Pin_4), U6.12 (O0)
- net VSEL: now also U15.1 (S), U16.1 (S), U17.1 (S)
- net VID9: now reaches J5.6 (Pin_6)
- net VID9: now also U15.3 (I1a)
- net A8: now reaches J5.7 (Pin_7)
- net A8: now also U15.14 (I0d)
- net VID8: now reaches J5.8 (Pin_8)
- net VID8: now also U15.13 (I1d)
- net S: now reaches J6.18 (Pin_18)
- net S: now also JVID.1 (Pin_1)
- net A12: now reaches J6.20 (Pin_20)
- net A12: now also U1.2 (A_{12})
- net at U6.15 (E): now also U6.7 (O3)
- net ~{RESET}: now reaches U1.26 (~{RESET})
- net ~{RESET}: now also JP1.1 (A), U11.10 (~{S}), U13.6
- net A15: now reaches U1.5 (A_{15})
- net A15: now also U14.1
- new net: C6.1, R4.2, U12.11 (R/Cext)
- new net: C6.2, U12.10 (Cext)
- new net: U14.11, U6.2 (A0)
- new net: U14.3, U6.3 (A1)
- new net: C25.2, R3.1, U13.13
- new net: U11.3 (C), U13.2
- new net: U11.11 (C), U12.6 (Q), U13.5
- new net: JP1.2 (B), U13.12
- new net: U11.5 (Q), U12.5 (B)
- new net EO: U11.9 (Q), U14.12, U14.2, U14.4
- new net G: JVID.2 (Pin_2)
- new net MQ: U14.10, U6.1 (E), U9.5
- new net S1: U11.1 (~{R})
- no-connect marks 0 -> 5
Other:
- note added: "Non si vede dove va, sembra quasi scollegato. Da misurare ---->"
- note added: "Questo è il break della tastiera DIRETTO!"
- note added: "Qui ci vanno le uscite di U15 U16 U17"
- moved on the sheet: J10, J6
